File: NG_IMU_Shield_Board/NG_IMU_Shield_Board.kicad_sch (KiCad schematic)
At the start: 20 parts, among them J1 Conn_01x04_Female, J2 Conn_01x02_Male, J3 Conn_01x10_Female, J4 Conn_01x03_Female, J5 Conn_02x12_Top_Bottom, J6 Conn_01x11_Male, U1 SN75LBC175, U2 Level_Converter, U3 Teensy_v4.0

Commit message: Added datasheets/etc. and cleanup
Parts:
- removed unit 3 of U1
- added unit 3 of U1
- U1: symbol NG_IMU_Shield_Board:SN75ALS175 -> NG_IMU_Shield_Board:SN75LBC175
Connections:
- net +5V: now also U1.16 (V+)
- net 0V: now also U1.8 (V-)
Changed lines of the file:
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@@
       (effects (font (size 1.27 1.27)) hide)
     )
-    (property "Datasheet" "" (id 3) (at 139.7 99.06 0)
+    (property "Datasheet" "https://www.pjrc.com/store/teensy40.html" (id 3) (at 139.7 99.06 0)
       (effects (font (size 1.27 1.27)) hide)
     )
@@
       (effects (font (size 1.27 1.27)) hide)
     )
-    (property "Datasheet" "" (id 3) (at 104.14 88.9 0)
+    (property "Datasheet" "https://www.sparkfun.com/products/12009" (id 3) (at 104.14 88.9 0)
       (effects (font (size 1.27 1.27)) hide)
     )
@@
     (pin "2")
   )
-  (symbol (lib_id "NG_IMU_Shield_Board:SN75ALS175") (at 64.77 124.46 0) (unit 2)
+  (symbol (lib_id "NG_IMU_Shield_Board:SN75LBC175") (at 104.14 135.89 0) (mirror x) (unit 3)
+    (in_bom yes) (on_board yes) (fields_autoplaced)
+    (property "Reference" "U1" (id 0) (at 100.9651 134.9815 0)
+      (effects (font (size 1.27 1.27)) (justify right))
+    )
+    (property "Value" "SN75LBC175" (id 1) (at 100.9651 137.7566 0)
+      (effects (font (size 1.27 1.27)) (justify right))
+    )
+    (property "Footprint" "Package_SO:SOIC-16_3.9x9.9mm_P1.27mm" (id 2) (at 104.14 135.89 0)
+      (effects (font (size 1.27 1.27)) hide)
+    )
+    (property "Datasheet" "https://www.ti.com/lit/ds/symlink/sn75lbc175a.pdf" (id 3) (at 104.14 135.89 0)
+      (effects (font (size 1.27 1.27)) hide)
+    )
+    (pin "16")
+    (pin "8")
+  )
+  (symbol (lib_id "NG_IMU_Shield_Board:SN75LBC175") (at 64.77 124.46 0) (unit 2)
     (in_bom yes) (on_board yes) (fields_autoplaced)
     (property "Reference" "U1" (id 0) (at 64.77 109.1905 0))
@@
       (effects (font (size 1.27 1.27)) hide)
     )
-    (property "Datasheet" "" (id 3) (at 64.77 124.46 0)
+    (property "Datasheet" "https://www.ti.com/lit/ds/symlink/sn75lbc175a.pdf" (id 3) (at 64.77 124.46 0)
       (effects (font (size 1.27 1.27)) hide)
     )
@@
     (pin "2")
   )
-  (symbol (lib_id "NG_IMU_Shield_Board:SN75ALS175") (at 104.14 135.89 0) (mirror x) (unit 3)
-    (in_bom yes) (on_board yes) (fields_autoplaced)
-    (property "Reference" "U1" (id 0) (at 100.9651 134.9815 0)
-      (effects (font (size 1.27 1.27)) (justify right))
-    )
-    (property "Value" "SN75LBC175" (id 1) (at 100.9651 137.7566 0)
-      (effects (font (size 1.27 1.27)) (justify right))
-    )
-    (property "Footprint" "Package_SO:SOIC-16_3.9x9.9mm_P1.27mm" (id 2) (at 104.14 135.89 0)
-      (effects (font (size 1.27 1.27)) hide)
-    )
-    (property "Datasheet" "" (id 3) (at 104.14 135.89 0)
-      (effects (font (size 1.27 1.27)) hide)
-    )
-    (pin "16")
-    (pin "8")
-  )
   (symbol (lib_id "Device:LED_GABR") (at 185.42 43.18 180) (unit 1)
     (in_bom yes) (on_board yes)
@@
     (pin "9")
   )
-  (symbol (lib_id "NG_IMU_Shield_Board:SN75ALS175") (at 64.77 93.98 0) (unit 1)
+  (symbol (lib_id "NG_IMU_Shield_Board:SN75LBC175") (at 64.77 93.98 0) (unit 1)
     (in_bom yes) (on_board yes) (fields_autoplaced)
     (property "Reference" "U1" (id 0) (at 64.77 78.7105 0))
@@
       (effects (font (size 1.27 1.27)) hide)
     )
-    (property "Datasheet" "" (id 3) (at 64.77 93.98 0)
+    (property "Datasheet" "https://www.ti.com/lit/ds/symlink/sn75lbc175a.pdf" (id 3) (at 64.77 93.98 0)
       (effects (font (size 1.27 1.27)) hide)
     )
@@
       (reference "U1") (unit 2) (value "SN75LBC175") (footprint "Package_SO:SOIC-16_3.9x9.9mm_P1.27mm")
     )
-    (path "/98cea5c7-b520-4360-90a2-00904ee27b87"
+    (path "/7831b541-e0d2-4aeb-b1b4-806d32aaad20"
       (reference "U1") (unit 3) (value "SN75LBC175") (footprint "Package_SO:SOIC-16_3.9x9.9mm_P1.27mm")
     )
