File: NG_IMU_Shield_Board/NG_IMU_Shield_Board.kicad_sch (KiCad schematic)
At the start: 20 parts, among them J1 Conn_01x04_Female, J2 Conn_01x02_Male, J3 Conn_01x10_Female, J4 Conn_01x03_Female, J5 Conn_02x12_Top_Bottom, J6 Conn_01x11_Male, U1 SN75LBC175, U2 Level_Converter, U3 Teensy_v4.0

Commit message: Moved board to match original coordinates, added CTRL, and minor changes
Parts:
- added J8: Conn_01x01_Female, Connector_PinSocket_2.54mm:PinSocket_1x01_P2.54mm_Vertical, symbol Connector:Conn_01x01_Female
- R1: footprint Resistor_SMD:R_0805_2012Metric_Pad1.20x1.40mm_HandSolder -> Resistor_SMD:R_1206_3216Metric_Pad1.30x1.75mm_HandSolder
Connections:
- new net CTRL: J8.1 (Pin_1)
Changed lines of the file:
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@@
     (effects (font (size 2.0066 2.0066)) (justify right bottom))
+  )
+  (label "CTRL" (at 181.61 76.2 180)
+    (effects (font (size 1.524 1.524)) (justify right bottom))
   )
   (label "G1" (at 215.9 88.9 180)
@@
     (property "Reference" "R1" (id 0) (at 222.25 40.132 90))
     (property "Value" "220" (id 1) (at 222.25 38.1 90))
-    (property "Footprint" "Resistor_SMD:R_0805_2012Metric_Pad1.20x1.40mm_HandSolder" (id 2) (at 222.25 36.322 90)
+    (property "Footprint" "Resistor_SMD:R_1206_3216Metric_Pad1.30x1.75mm_HandSolder" (id 2) (at 222.25 36.322 90)
       (effects (font (size 1.27 1.27)) hide)
     )
@@
     (pin "2")
   )
+  (symbol (lib_id "Connector:Conn_01x01_Female") (at 186.69 76.2 0) (unit 1)
+    (in_bom yes) (on_board yes) (fields_autoplaced)
+    (property "Reference" "J8" (id 0) (at 187.4012 75.2915 0)
+      (effects (font (size 1.27 1.27)) (justify left))
+    )
+    (property "Value" "Conn_01x01_Female" (id 1) (at 187.4012 78.0666 0)
+      (effects (font (size 1.27 1.27)) (justify left))
+    )
+    (property "Footprint" "Connector_PinSocket_2.54mm:PinSocket_1x01_P2.54mm_Vertical" (id 2) (at 186.69 76.2 0)
+      (effects (font (size 1.27 1.27)) hide)
+    )
+    (property "Datasheet" "~" (id 3) (at 186.69 76.2 0)
+      (effects (font (size 1.27 1.27)) hide)
+    )
+    (pin "1")
+  )
   (symbol (lib_id "NG_IMU_Interface_Board-rescue:R") (at 196.85 48.26 90) (unit 1)
     (in_bom yes) (on_board yes)
@@
       (reference "J6") (unit 1) (value "Conn_01x11_Male") (footprint "Connector_PinHeader_2.54mm:PinHeader_1x11_P2.54mm_Vertical")
     )
+    (path "/b3d89762-54ee-4dc0-8c86-98a5d2a2dca5"
+      (reference "J8") (unit 1) (value "Conn_01x01_Female") (footprint "Connector_PinSocket_2.54mm:PinSocket_1x01_P2.54mm_Vertical")
+    )
     (path "/afee99b0-6a90-4948-bc99-81059c1d912b"
       (reference "JP1") (unit 1) (value "Jumper_2_Open") (footprint "Connector_PinHeader_2.54mm:PinHeader_1x02_P2.54mm_Vertical")
     )
     (path "/00000000-0000-0000-0000-00005acac33c"
-      (reference "R1") (unit 1) (value "220") (footprint "Resistor_SMD:R_0805_2012Metric_Pad1.20x1.40mm_HandSolder")
+      (reference "R1") (unit 1) (value "220") (footprint "Resistor_SMD:R_1206_3216Metric_Pad1.30x1.75mm_HandSolder")
     )
     (path "/ceb6cdcb-8e0b-4367-b390-08e19d41682c"

Commit message: Added pin socket to allow disabling power with a jumper
Parts:
- J8: value Conn_01x01_Female -> Conn_01x02_Female; footprint Connector_PinSocket_2.54mm:PinSocket_1x01_P2.54mm_Vertical -> Connector_PinSocket_2.54mm:PinSocket_1x02_P2.54mm_Vertical; symbol Connector:Conn_01x01_Female -> Connector:Conn_01x02_Female
Connections:
- net 0V: now also J8.2 (Pin_2)
Changed lines of the file:
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@@
+    (effects (font (size 1.524 1.524)) (justify right bottom))
+  )
+  (label "0V" (at 181.61 78.74 180)
     (effects (font (size 1.524 1.524)) (justify right bottom))
   )
@@
     (pin "2")
   )
-  (symbol (lib_id "Connector:Conn_01x01_Female") (at 186.69 76.2 0) (unit 1)
+  (symbol (lib_id "Connector:Conn_01x02_Female") (at 186.69 76.2 0) (unit 1)
     (in_bom yes) (on_board yes) (fields_autoplaced)
     (property "Reference" "J8" (id 0) (at 187.4012 75.2915 0)
       (effects (font (size 1.27 1.27)) (justify left))
     )
-    (property "Value" "Conn_01x01_Female" (id 1) (at 187.4012 78.0666 0)
-      (effects (font (size 1.27 1.27)) (justify left))
-    )
-    (property "Footprint" "Connector_PinSocket_2.54mm:PinSocket_1x01_P2.54mm_Vertical" (id 2) (at 186.69 76.2 0)
+    (property "Value" "Conn_01x02_Female" (id 1) (at 187.4012 78.0666 0)
+      (effects (font (size 1.27 1.27)) (justify left))
+    )
+    (property "Footprint" "Connector_PinSocket_2.54mm:PinSocket_1x02_P2.54mm_Vertical" (id 2) (at 186.69 76.2 0)
       (effects (font (size 1.27 1.27)) hide)
     )
@@
     )
     (pin "1")
+    (pin "2")
   )
   (symbol (lib_id "NG_IMU_Interface_Board-rescue:R") (at 196.85 48.26 90) (unit 1)
@@
     )
     (path "/b3d89762-54ee-4dc0-8c86-98a5d2a2dca5"
-      (reference "J8") (unit 1) (value "Conn_01x01_Female") (footprint "Connector_PinSocket_2.54mm:PinSocket_1x01_P2.54mm_Vertical")
+      (reference "J8") (unit 1) (value "Conn_01x02_Female") (footprint "Connector_PinSocket_2.54mm:PinSocket_1x02_P2.54mm_Vertical")
     )
     (path "/afee99b0-6a90-4948-bc99-81059c1d912b"
